File: sesame.sch (KiCad schematic (older format))
At the start: 155 parts, among them U1 ATmega32A-PU

Commit message: Change to Mini USB
Parts:
- removed AVR1: Conn_01x06, Connector_PinHeader_2.54mm:PinHeader_1x06_P2.54mm_Vertical, symbol Connector_Generic:Conn_01x06
- removed R4, R5: 5.1K, Resistor_THT:R_Axial_DIN0207_L6.3mm_D2.5mm_P10.16mm_Horizontal, symbol Device:R
- removed USB1: USB_C_Receptacle_USB2.0, custom_parts:USB_C_GCT_USB4085, symbol Connector:USB_C_Receptacle_USB2.0
- added AVR1: Conn_02x03_Odd_Even, Connector_PinHeader_2.54mm:PinHeader_2x03_P2.54mm_Vertical, symbol Connector_Generic:Conn_02x03_Odd_Even
- added USB1: USB_B_Mini, Keebio-Parts:USB-Mini-B_ LCSC-C46398, symbol Connector:USB_B_Mini
- MX1, MX10, MX11, MX12, MX13, MX14, MX15, MX16, MX17, MX18, MX19, MX2, MX20, MX21, MX22, MX23, MX24, MX25, MX26, MX27, MX28, MX29, MX3, MX30, MX31, MX32, MX33, MX34, MX35, MX36, MX37, MX38, MX39, MX4, MX40, MX41, MX42, MX43, MX44, MX45, MX46, MX47, MX48, MX49, MX5, MX50, MX51, MX52, MX53, MX54, MX55, MX56, MX57, MX58, MX59, MX6, MX60, MX61, MX62, MX63, MX64, MX65, MX66, MX67, MX68, MX69, MX7, MX8, MX9: symbol MX_Alps_Hybrid:MX-NoLED -> sesame-rescue:MX-NoLED-MX_Alps_Hybrid
Connections:
- wire segments 231 -> 230
- no-connect marks 0 -> 1
